File: 3v.kicad_sch (KiCad schematic)
At the start: 4 parts, among them U1 AMS1117-3.3

Commit message: Minor updates to HW Rev 1.0
Parts:
- C4, C5: footprint LIBS:C_Radial -> LIBS:CT_3528
Changed lines of the file:
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@@
 			)
 		)
-		(property "Footprint" "LIBS:C_Radial"
+		(property "Footprint" "LIBS:CT_3528"
 			(at 69.85 41.91 0)
 			(effects
@@
 			)
 		)
-		(property "Footprint" "LIBS:C_Radial"
+		(property "Footprint" "LIBS:CT_3528"
 			(at 30.48 41.91 0)
 			(effects
