File: valera.kicad_pcb (KiCad board)
At the start: 2 copper layers, 85.6 x 54 mm, 89 parts, among them J1 Audio Jumpers, J2 PWM Jumper, J3 JOY-1, Q1 BC850, Q2 BC850, Q3 BC850, Q4 BC850, U1 AMS1117-3.3, U2 TDA1387T

Commit message: Minor updates to HW Rev 1.0
Parts:
- added C18: 10u, LIBS:C_0805, F.Cu at (226.0, 67.0)
- added R41: 5.1K, LIBS:R_0805, F.Cu at (226.0, 75.0)
- added R42: 5.1K, LIBS:R_0805, F.Cu at (226.0, 71.0)
- added USB1: USB Type C, LIBS:USB-TYPE-C-31-M-12_lib2, F.Cu at (237.4, 70.9)
- C12, C4, C5, C6, C7: footprint LIBS:C_Radial -> LIBS:CT_3528
- moved U1 6.40 mm to (218.5, 70.0), turned to 180 degrees
- moved C7 3.28 mm to (208.2, 53.8), turned to 90 degrees
- moved JP1 2.64 mm to (221.3, 75.0)
- moved C6 1.39 mm to (203.6, 53.8), turned to 90 degrees
- moved C5 1.00 mm to (224.8, 86.0), turned to 0 degrees
- moved C12 0.92 mm to (199.0, 53.8), turned to 90 degrees
- moved C4 0.70 mm to (216.6, 86.0), turned to 180 degrees
Connections:
- net /Pico2/GPIO23_1 renamed /Pico2/GPIO23
- net /Pico2/GPIO8_1 renamed /Pico2/GPIO8
- net /Pico2/RUN_1 renamed /Pico2/RUN
Routing:
- net VBUS: track 228.9 -> 251.9 mm
- net /Tape Loader/LOAD_IN: track 64.4 -> 73.6 mm
- net GND: track 0.00 -> 5.41 mm, vias 26 -> 30
- net Net-(USB1-CC1): track 0.00 -> 4.45 mm
- net Net-(USB1-CC2): track 0.00 -> 4.16 mm
- net +3V3: track 165.6 -> 169.6 mm, vias 6 -> 4
- net /SD_MISO: track 66.6 -> 70.6 mm
- net /Audio Out/L: track 22.1 -> 18.6 mm, vias 0 -> 1
- net /Audio Out/+5VA: track 102.8 -> 99.5 mm, vias 3 -> 4
- net /Power/D+: track 0.00 -> 3.00 mm
- net /Power/D-: track 0.00 -> 3.00 mm
- net Net-(Q3-C): track 73.0 -> 70.0 mm
- net /3V3_EXT: track 5.37 -> 6.99 mm
- net /Gamepad/J1_DATA: track 135.4 -> 134.0 mm
- net Net-(Q4-C): track 42.4 -> 42.5 mm, vias 1 -> 2
Other:
- board text added: "M2 RP2350"
- board text added: "Power"
- board text removed: "RP2350 PICO2"
