File: valera.kicad_sch (KiCad schematic)
At the start: 6 parts, among them J1 Audio Jumpers, J2 PWM Jumper

Commit message: Minor updates to HW Rev 1.0
Connections:
- no-connect marks 6 -> 8
Other:
- added sheet Power (power.kicad_sch)
Changed lines of the file:
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@@
+	)
+	(no_connect
+		(at 54.61 162.56)
+	)
+	(no_connect
+		(at 54.61 160.02)
 	)
 	(no_connect
@@
 				)
 			)
+		)
+	)
+	(sheet
+		(at 54.61 157.48)
+		(size 13.97 7.62)
+		(fields_autoplaced yes)
+		(stroke
+			(width 0.1524)
+			(type solid)
+		)
+		(fill
+			(color 0 0 0 0.0000)
+		)
+		(property "Sheetname" "Power"
+			(at 54.61 156.7684 0)
+			(effects
+				(font
+					(size 1.27 1.27)
+				)
+				(justify left bottom)
+			)
+		)
+		(property "Sheetfile" "power.kicad_sch"
+			(at 54.61 165.6846 0)
+			(effects
+				(font
+					(size 1.27 1.27)
+				)
+				(justify left top)
+				(hide yes)
+			)
+		)
+		(pin "D-" input
+			(at 54.61 160.02 180)
+			(effects
+				(font
+					(size 1.27 1.27)
+				)
+				(justify left)
+			)
+		)
+		(pin "D+" input
+			(at 54.61 162.56 180)
+			(effects
+				(font
+					(size 1.27 1.27)
+				)
+				(justify left)
+			)
+		)
+		(instances
+			(project "valera"
+				(path "/621f55f1-01af-437d-a2cb-120cc66267c2"
+					(page "10")
+				)
+			)
