File: audio_out.kicad_sch (KiCad schematic)
At the start: 34 parts, among them Q3 BC850, Q4 BC850, U2 TDA1387T

Commit message: Minor updates to HW Rev 1.0
Parts:
- C12, C6, C7: footprint LIBS:C_Radial -> LIBS:CT_3528
Changed lines of the file:
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@@
 			)
 		)
-		(property "Footprint" "LIBS:C_Radial"
+		(property "Footprint" "LIBS:CT_3528"
 			(at 99.06 40.64 0)
 			(effects
@@
 			)
 		)
-		(property "Footprint" "LIBS:C_Radial"
+		(property "Footprint" "LIBS:CT_3528"
 			(at 208.28 93.98 0)
 			(effects
@@
 			)
 		)
-		(property "Footprint" "LIBS:C_Radial"
+		(property "Footprint" "LIBS:CT_3528"
 			(at 208.28 46.99 0)
 			(effects

Commit message: Minor updates to schematics
Other:
- note removed: "GP_10"
- note removed: "GP_11"
- note removed: "GP_9"
Changed lines of the file:
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@@
-		)
-	)
-	(text "GP_10"
-		(exclude_from_sim no)
-		(at 239.014 58.674 0)
-		(effects
-			(font
-				(size 1.27 1.27)
-			)
-		)
-	)
-	(text "GP_11"
-		(exclude_from_sim no)
-		(at 238.76 105.41 0)
-		(effects
-			(font
-				(size 1.27 1.27)
-			)
-		)
-	)
-	(text "GP_9"
-		(exclude_from_sim no)
-		(at 238.76 113.03 0)
-		(effects
-			(font
-				(size 1.27 1.27)
-			)
-		)
-	)
-	(text "GP_9"
-		(exclude_from_sim no)
-		(at 238.76 66.04 0)
-		(effects
-			(font
-				(size 1.27 1.27)
-			)
 		)
 	)
