File: hdmi.kicad_sch (KiCad schematic)
At the start: 10 parts

Commit message: Minor updates to schematics
Other:
- note removed: "GP_12"
- note removed: "GP_13"
- note removed: "GP_14"
- note removed: "GP_15"
- note removed: "GP_16"
- note removed: "GP_17"
- note removed: "GP_18"
- note removed: "GP_19"
Changed lines of the file:
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@@
-		)
-	)
-	(text "GP_14"
-		(exclude_from_sim no)
-		(at 119.888 95.758 0)
-		(effects
-			(font
-				(size 1.27 1.27)
-			)
-		)
-	)
-	(text "GP_16"
-		(exclude_from_sim no)
-		(at 119.888 103.378 0)
-		(effects
-			(font
-				(size 1.27 1.27)
-			)
-		)
-	)
-	(text "GP_18"
-		(exclude_from_sim no)
-		(at 120.142 110.998 0)
-		(effects
-			(font
-				(size 1.27 1.27)
-			)
-		)
-	)
-	(text "GP_17"
-		(exclude_from_sim no)
-		(at 120.142 108.458 0)
-		(effects
-			(font
-				(size 1.27 1.27)
-			)
-		)
-	)
-	(text "GP_19"
-		(exclude_from_sim no)
-		(at 120.142 116.078 0)
-		(effects
-			(font
-				(size 1.27 1.27)
-			)
-		)
-	)
-	(text "GP_13"
-		(exclude_from_sim no)
-		(at 119.888 93.218 0)
-		(effects
-			(font
-				(size 1.27 1.27)
-			)
-		)
-	)
-	(text "GP_15"
-		(exclude_from_sim no)
-		(at 119.888 100.838 0)
-		(effects
-			(font
-				(size 1.27 1.27)
-			)
-		)
-	)
-	(text "GP_12"
-		(exclude_from_sim no)
-		(at 120.142 88.138 0)
-		(effects
-			(font
-				(size 1.27 1.27)
-			)
 		)
 	)
