File: microsd.kicad_sch (KiCad schematic)
At the start: 2 parts

Commit message: Minor updates to schematics
Other:
- note removed: "GP_4"
- note removed: "GP_5"
- note removed: "GP_6"
- note removed: "GP_7"
Changed lines of the file:
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@@
-		)
-	)
-	(text "GP_6"
-		(exclude_from_sim no)
-		(at 68.58 60.198 0)
-		(effects
-			(font
-				(size 1.27 1.27)
-			)
-		)
-	)
-	(text "GP_5"
-		(exclude_from_sim no)
-		(at 68.58 52.578 0)
-		(effects
-			(font
-				(size 1.27 1.27)
-			)
-		)
-	)
-	(text "GP_7"
-		(exclude_from_sim no)
-		(at 68.58 55.118 0)
-		(effects
-			(font
-				(size 1.27 1.27)
-			)
-		)
-	)
-	(text "GP_4"
-		(exclude_from_sim no)
-		(at 68.58 65.278 0)
-		(effects
-			(font
-				(size 1.27 1.27)
-			)
 		)
 	)
