File: ps2.kicad_sch (KiCad schematic)
At the start: 14 parts

Commit message: Minor updates to schematics
Other:
- note removed: "KB_CLK_3V"
- note removed: "KB_DATA_3V"
Changed lines of the file:
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@@
-		)
-	)
-	(text "KB_DATA_3V"
-		(exclude_from_sim no)
-		(at 131.064 72.39 0)
-		(effects
-			(font
-				(size 1.27 1.27)
-			)
-		)
-	)
-	(text "KB_CLK_3V"
-		(exclude_from_sim no)
-		(at 131.572 67.564 0)
-		(effects
-			(font
-				(size 1.27 1.27)
-			)
 		)
 	)
